File: robot_principal/electronique/Carte_puissance/Carte_puissance.kicad_sch (KiCad schematic)
At the start: 14 parts, among them J1 Conn_01x02, J10 Conn_01x04, J2 Conn_01x02, J3 Conn_01x02, J4 Screw_Terminal_01x02, J5 Screw_Terminal_01x02, J6 Screw_Terminal_01x02, J7 Conn_01x04, J8 Conn_01x04, J9 Conn_01x04

Commit message: carte elec de puissance terminée
Parts:
- removed J10, J7, J8, J9: Conn_01x04, symbol Connector_Generic:Conn_01x04
- removed J2, J3: Conn_01x02, symbol Connector_Generic:Conn_01x02
- removed J4, J5, J6: Screw_Terminal_01x02, symbol Connector:Screw_Terminal_01x02
- added C1, C2, C3, C4: C_Polarized, Capacitor_THT:CP_Radial_D10.0mm_P5.00mm, symbol Device:C_Polarized
- added F1: Fuse, Fuse:FuseHolder_Blade_ATO_Littelfuse_FLR_178.6165, symbol Device:Fuse
- added H1, H2, H3, H4: MountingHole, MountingHole:MountingHole_3.2mm_M3, symbol Mechanical:MountingHole
- added J10, J7, J8, J9: Conn_01x06, Connector_JST:JST_XH_B6B-XH-A_1x06_P2.50mm_Vertical, symbol Connector_Generic:Conn_01x06
- added J13, J14, J15, J16, J17, J18, J19, J20, J28, J29: Conn_01x02, Connector_PinHeader_2.54mm:PinHeader_1x02_P2.54mm_Vertical, symbol Connector_Generic:Conn_01x02
- added J2: Screw_Terminal_01x10, TerminalBlock_Phoenix:TerminalBlock_Phoenix_MKDS-1,5-10-5.08_1x10_P5.08mm_Horizontal, symbol Connector:Screw_Terminal_01x10
- added J21, J22, J23, J24, J31, J32: Conn_01x04, Connector_PinHeader_2.54mm:PinHeader_1x04_P2.54mm_Vertical, symbol Connector_Generic:Conn_01x04
- added J25: Screw_Terminal_01x02, TerminalBlock_Phoenix:TerminalBlock_Phoenix_MKDS-1,5-2-5.08_1x02_P5.08mm_Horizontal, symbol Connector:Screw_Terminal_01x02
- added J27: Conn_01x06, Connector_PinHeader_2.54mm:PinHeader_1x06_P2.54mm_Vertical, symbol Connector_Generic:Conn_01x06
- added J30: Screw_Terminal_01x06, TerminalBlock_Phoenix:TerminalBlock_Phoenix_MKDS-1,5-6-5.08_1x06_P5.08mm_Horizontal, symbol Connector:Screw_Terminal_01x06
- J1: footprint (none) -> Connector_AMASS:AMASS_XT60-M_1x02_P7.20mm_Vertical
Connections:
- net +24V: now also F1.1, J30.1 (Pin_1), J30.2 (Pin_2); no longer J1.1 (Pin_1)
- net +3.3V: now also J13.1 (Pin_1), J14.1 (Pin_1), J15.1 (Pin_1), J16.1 (Pin_1), J17.1 (Pin_1), J18.1 (Pin_1), J19.1 (Pin_1), J20.1 (Pin_1), J28.1 (Pin_1), J29.1 (Pin_1)
- net Alim_22.2V: now also C1.1, C2.1, C3.1, C4.1, J2.6 (Pin_6), J2.7 (Pin_7), J2.9 (Pin_9), J30.3 (Pin_3)
- net GND: now also C1.2, C2.2, C3.2, C4.2, J2.10 (Pin_10), J2.2 (Pin_2), J2.3 (Pin_3), J2.5 (Pin_5), J2.8 (Pin_8), J21.4 (Pin_4), J22.4 (Pin_4), J23.4 (Pin_4), J24.4 (Pin_4), J25.1 (Pin_1), J27.1 (Pin_1), J27.2 (Pin_2), J27.3 (Pin_3), J27.4 (Pin_4), J27.5 (Pin_5), J27.6 (Pin_6), J28.2 (Pin_2), J30.4 (Pin_4), J30.5 (Pin_5)
- net at A2.3 (1B): now also J7.1 (Pin_1)
- net at A2.4 (1A): now also J7.3 (Pin_3)
- net at A2.5 (2A): now also J7.4 (Pin_4)
- net at A2.6 (2B): now also J7.6 (Pin_6)
- net at A3.3 (1B): now also J9.1 (Pin_1)
- net at A3.4 (1A): now also J9.3 (Pin_3)
- net at A3.5 (2A): now also J9.4 (Pin_4)
- net at A3.6 (2B): now also J9.6 (Pin_6)
- net at A3.10 (MS1): now also J15.2 (Pin_2)
- net at A3.11 (MS2): now also J16.2 (Pin_2)
- net at A3.13 (~{RESET}): no longer A3.14 (~{SLEEP})
- net at A3.15 (STEP): now also J23.1 (Pin_1)
- net at A3.16 (DIR): now also J23.2 (Pin_2)
- net at A3.9 (~{ENABLE}): now also J23.3 (Pin_3)
- net at A1.3 (1B): now also J10.1 (Pin_1)
- net at A1.4 (1A): now also J10.3 (Pin_3)
- net at A1.5 (2A): now also J10.4 (Pin_4)
- net at A1.6 (2B): now also J10.6 (Pin_6)
- net at A4.10 (MS1): now also J17.2 (Pin_2)
- net at A4.11 (MS2): now also J18.2 (Pin_2)
- net at A4.13 (~{RESET}): no longer A4.14 (~{SLEEP})
- net at A4.15 (STEP): now also J22.1 (Pin_1)
- net at A4.16 (DIR): now also J22.2 (Pin_2)
- net at A4.3 (1B): now also J8.1 (Pin_1)
- net at A4.4 (1A): now also J8.3 (Pin_3)
- net at A4.5 (2A): now also J8.4 (Pin_4)
- net at A4.6 (2B): now also J8.6 (Pin_6)
- net at A4.9 (~{ENABLE}): now also J22.3 (Pin_3)
- net at A1.10 (MS1): now also J19.2 (Pin_2)
- net at A1.11 (MS2): now also J20.2 (Pin_2)
- net at A1.12 (MS3): now also J29.2 (Pin_2)
- net at A1.15 (STEP): now also J24.1 (Pin_1)
- net at A1.16 (DIR): now also J24.2 (Pin_2)
- net at A1.9 (~{ENABLE}): now also J24.3 (Pin_3)
- net at A2.10 (MS1): now also J13.2 (Pin_2)
- net at A2.11 (MS2): now also J14.2 (Pin_2)
- net at A2.13 (~{RESET}): no longer A2.14 (~{SLEEP})
- net at A2.15 (STEP): now also J21.1 (Pin_1)
- net at A2.16 (DIR): now also J21.2 (Pin_2)
- net at A2.9 (~{ENABLE}): now also J21.3 (Pin_3)
- new net ALIM: F1.2, J1.1 (Pin_1), J25.2 (Pin_2)
- new net Logique_+5V: J2.1 (Pin_1), J30.6 (Pin_6), J32.1 (Pin_1), J32.2 (Pin_2), J32.3 (Pin_3), J32.4 (Pin_4)
- new net actio_+6V: J2.4 (Pin_4), J31.1 (Pin_1), J31.2 (Pin_2), J31.3 (Pin_3), J31.4 (Pin_4)
Other:
- moved on the sheet: A1, A2, A3, A4, J1
